File: 2xVCA_SMD.sch (EAGLE design)
At the start: 50 parts, among them IC1 TL072D, IC2 LM13700M, IC3 TL072D, Q1 MMBT3906LT1SMD, Q2 MMBT3906LT1SMD, Q4 BC847SMD, Q5 BC847SMD

Commit message: Fixed component labels. Minor routing adjustments. Spread PSU components a bit. Added board type label & copyright notice.
Parts:
- C1, C10, C3, C5, C6, C7, C8, C9: device rcl:C-EUC0603 -> rcl:C-EUC0603K
Changed lines of the file:
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@@
 <part name="GND2" library="supply1" deviceset="GND" device=""/>
 <part name="P+1" library="supply1" deviceset="VCC" device=""/>
-<part name="C1" library="rcl" deviceset="C-EU" device="C0603" value="470p"/>
+<part name="C1" library="rcl" deviceset="C-EU" device="C0603K" value="470p"/>
 <part name="R4" library="rcl" deviceset="R-EU_" device="R0603" value="47k"/>
 <part name="GND3" library="supply1" deviceset="GND" device=""/>
@@
 <part name="GND15" library="supply1" deviceset="GND" device=""/>
 <part name="GND16" library="supply1" deviceset="GND" device=""/>
-<part name="C5" library="rcl" deviceset="C-EU" device="C0603" value="100n"/>
+<part name="C5" library="rcl" deviceset="C-EU" device="C0603K" value="100n"/>
 <part name="GND17" library="supply1" deviceset="GND" device=""/>
 <part name="P+3" library="supply1" deviceset="VCC" device=""/>
@@
 <part name="R11" library="rcl" deviceset="R-EU_" device="R0603" value="33k"/>
 <part name="R12" library="rcl" deviceset="R-EU_" device="R0603" value="47k"/>
-<part name="C3" library="rcl" deviceset="C-EU" device="C0603" value="470p"/>
+<part name="C3" library="rcl" deviceset="C-EU" device="C0603K" value="470p"/>
 <part name="Q1" library="transistor-pnp" deviceset="MMBT3906*" device="SMD" technology="LT1"/>
 <part name="R13" library="rcl" deviceset="R-EU_" device="R0603" value="100k"/>
@@
 <part name="R15" library="rcl" deviceset="R-EU_" device="R0603" value="100k"/>
 <part name="R16" library="rcl" deviceset="R-EU_" device="R0603" value="220"/>
-<part name="C6" library="rcl" deviceset="C-EU" device="C0603" value="100n"/>
-<part name="C7" library="rcl" deviceset="C-EU" device="C0603" value="100n"/>
-<part name="C8" library="rcl" deviceset="C-EU" device="C0603" value="100n"/>
-<part name="C9" library="rcl" deviceset="C-EU" device="C0603" value="100n"/>
-<part name="C10" library="rcl" deviceset="C-EU" device="C0603" value="100n"/>
+<part name="C6" library="rcl" deviceset="C-EU" device="C0603K" value="100n"/>
+<part name="C7" library="rcl" deviceset="C-EU" device="C0603K" value="100n"/>
+<part name="C8" library="rcl" deviceset="C-EU" device="C0603K" value="100n"/>
+<part name="C9" library="rcl" deviceset="C-EU" device="C0603K" value="100n"/>
+<part name="C10" library="rcl" deviceset="C-EU" device="C0603K" value="100n"/>
 </parts>
 <sheets>
